Commit message: Cleaned up simulation environment

File: panda_description/urdf/panda.urdf.xacro (robot description, xacro)
@@ -91,4 +91,115 @@
     />
   </xacro:if>
+  <!-- ===== Static environment for open-loop chess ===== -->
+  <!-- Matches panda_description/worlds/tabletop_chess.sdf exactly -->
+  <link name="table_link">
+    <!-- Table top -->
+    <visual>
+      <origin xyz="0 0 0.25" rpy="0 0 0"/>
+      <geometry>
+        <box size="0.8 1.0 0.04"/>
+      </geometry>
+      <material name="table_top_mat">
+        <color rgba="0.6 0.4 0.2 1.0"/>
+      </material>
+    </visual>
+    <collision>
+      <origin xyz="0 0 0.25" rpy="0 0 0"/>
+      <geometry>
+        <box size="0.8 1.0 0.04"/>
+      </geometry>
+    </collision>
+    <!-- Leg 1 -->
+    <visual>
+      <origin xyz="0.35 0.45 0.115" rpy="0 0 0"/>
+      <geometry>
+        <box size="0.04 0.04 0.23"/>
+      </geometry>
+      <material name="table_leg_mat">
+        <color rgba="0.5 0.3 0.1 1.0"/>
+      </material>
+    </visual>
+    <collision>
+      <origin xyz="0.35 0.45 0.115" rpy="0 0 0"/>
+      <geometry>
+        <box size="0.04 0.04 0.23"/>
+      </geometry>
+    </collision>
+    <!-- Leg 2 -->
+    <visual>
+      <origin xyz="0.35 -0.45 0.115" rpy="0 0 0"/>
+      <geometry>
+        <box size="0.04 0.04 0.23"/>
+      </geometry>
+      <material name="table_leg_mat_2">
+        <color rgba="0.5 0.3 0.1 1.0"/>
+      </material>
+    </visual>
+    <collision>
+      <origin xyz="0.35 -0.45 0.115" rpy="0 0 0"/>
+      <geometry>
+        <box size="0.04 0.04 0.23"/>
+      </geometry>
+    </collision>
+    <!-- Leg 3 -->
+    <visual>
+      <origin xyz="-0.35 0.45 0.115" rpy="0 0 0"/>
+      <geometry>
+        <box size="0.04 0.04 0.23"/>
+      </geometry>
+      <material name="table_leg_mat_3">
+        <color rgba="0.5 0.3 0.1 1.0"/>
+      </material>
+    </visual>
+    <collision>
+      <origin xyz="-0.35 0.45 0.115" rpy="0 0 0"/>
+      <geometry>
+        <box size="0.04 0.04 0.23"/>
+      </geometry>
+    </collision>
+    <!-- Leg 4 -->
+    <visual>
+      <origin xyz="-0.35 -0.45 0.115" rpy="0 0 0"/>
+      <geometry>
+        <box size="0.04 0.04 0.23"/>
+      </geometry>
+      <material name="table_leg_mat_4">
+        <color rgba="0.5 0.3 0.1 1.0"/>
+      </material>
+    </visual>
+    <collision>
+      <origin xyz="-0.35 -0.45 0.115" rpy="0 0 0"/>
+      <geometry>
+        <box size="0.04 0.04 0.23"/>
+      </geometry>
+    </collision>
+  </link>
+  <joint name="world_to_table_joint" type="fixed">
+    <parent link="world"/>
+    <child link="table_link"/>
+    <origin xyz="0.6 0 0" rpy="0 0 0"/>
+  </joint>
+  <link name="chessboard_link">
+    <visual>
+      <origin xyz="0 0 0" rpy="0 0 0"/>
+      <geometry>
+        <box size="0.70 0.70 0.01"/>
+      </geometry>
+      <material name="chessboard_mat">
+        <color rgba="0.2 0.2 0.2 1.0"/>
+      </material>
+    </visual>
+    <collision>
+      <origin xyz="0 0 0" rpy="0 0 0"/>
+      <geometry>
+        <box size="0.70 0.70 0.01"/>
+      </geometry>
+    </collision>
+  </link>
+  <joint name="table_to_chessboard_joint" type="fixed">
+    <parent link="table_link"/>
+    <child link="chessboard_link"/>
+    <origin xyz="0 0 0.272" rpy="0 0 1.5708"/>
+  </joint>
   <!-- Gazebo - ROS 2 control -->
   <xacro:if value="$(arg ros2_control)">

Commit message: table

File: panda_description/urdf/panda.urdf.xacro (robot description, xacro)
@@ -95,6 +95,6 @@
   <link name="table_link">
     <!-- Table top -->
-    <visual>
-      <origin xyz="0 0 0.25" rpy="0 0 0"/>
+        <visual>
+      <origin xyz="0 0 0.16" rpy="0 0 0"/>
       <geometry>
         <box size="0.8 1.0 0.04"/>
@@ -105,5 +105,5 @@
     </visual>
     <collision>
-      <origin xyz="0 0 0.25" rpy="0 0 0"/>
+      <origin xyz="0 0 0.16" rpy="0 0 0"/>
       <geometry>
         <box size="0.8 1.0 0.04"/>
@@ -112,7 +112,7 @@
     <!-- Leg 1 -->
     <visual>
-      <origin xyz="0.35 0.45 0.115" rpy="0 0 0"/>
-      <geometry>
-        <box size="0.04 0.04 0.23"/>
+      <origin xyz="0.35 0.45 0.07" rpy="0 0 0"/>
+      <geometry>
+        <box size="0.04 0.04 0.14"/>
       </geometry>
       <material name="table_leg_mat">
@@ -121,14 +121,14 @@
     </visual>
     <collision>
-      <origin xyz="0.35 0.45 0.115" rpy="0 0 0"/>
-      <geometry>
-        <box size="0.04 0.04 0.23"/>
+      <origin xyz="0.35 0.45 0.07" rpy="0 0 0"/>
+      <geometry>
+        <box size="0.04 0.04 0.14"/>
       </geometry>
     </collision>
     <!-- Leg 2 -->
     <visual>
-      <origin xyz="0.35 -0.45 0.115" rpy="0 0 0"/>
-      <geometry>
-        <box size="0.04 0.04 0.23"/>
+      <origin xyz="0.35 -0.45 0.07" rpy="0 0 0"/>
+      <geometry>
+        <box size="0.04 0.04 0.14"/>
       </geometry>
       <material name="table_leg_mat_2">
@@ -137,14 +137,14 @@
     </visual>
     <collision>
-      <origin xyz="0.35 -0.45 0.115" rpy="0 0 0"/>
-      <geometry>
-        <box size="0.04 0.04 0.23"/>
+      <origin xyz="0.35 -0.45 0.07" rpy="0 0 0"/>
+      <geometry>
+        <box size="0.04 0.04 0.14"/>
       </geometry>
     </collision>
     <!-- Leg 3 -->
     <visual>
-      <origin xyz="-0.35 0.45 0.115" rpy="0 0 0"/>
-      <geometry>
-        <box size="0.04 0.04 0.23"/>
+      <origin xyz="-0.35 0.45 0.07" rpy="0 0 0"/>
+      <geometry>
+        <box size="0.04 0.04 0.14"/>
       </geometry>
       <material name="table_leg_mat_3">
@@ -153,14 +153,14 @@
     </visual>
     <collision>
-      <origin xyz="-0.35 0.45 0.115" rpy="0 0 0"/>
-      <geometry>
-        <box size="0.04 0.04 0.23"/>
+      <origin xyz="-0.35 0.45 0.07" rpy="0 0 0"/>
+      <geometry>
+        <box size="0.04 0.04 0.14"/>
       </geometry>
     </collision>
     <!-- Leg 4 -->
     <visual>
-      <origin xyz="-0.35 -0.45 0.115" rpy="0 0 0"/>
-      <geometry>
-        <box size="0.04 0.04 0.23"/>
+      <origin xyz="-0.35 -0.45 0.07" rpy="0 0 0"/>
+      <geometry>
+        <box size="0.04 0.04 0.14"/>
       </geometry>
       <material name="table_leg_mat_4">
@@ -169,16 +169,16 @@
     </visual>
     <collision>
-      <origin xyz="-0.35 -0.45 0.115" rpy="0 0 0"/>
-      <geometry>
-        <box size="0.04 0.04 0.23"/>
-      </geometry>
-    </collision>
-  </link>
-  <joint name="world_to_table_joint" type="fixed">
-    <parent link="world"/>
-    <child link="table_link"/>
-    <origin xyz="0.6 0 0" rpy="0 0 0"/>
-  </joint>
-  <link name="chessboard_link">
+      <origin xyz="-0.35 -0.45 0.07" rpy="0 0 0"/>
+      <geometry>
+        <box size="0.04 0.04 0.14"/>
+      </geometry>
+    </collision>
+    </link>
+    <joint name="world_to_table_joint" type="fixed">
+      <parent link="world"/>
+      <child link="table_link"/>
+      <origin xyz="0.6 0 0" rpy="0 0 0"/>
+    </joint>
+    <link name="chessboard_link">
     <visual>
       <origin xyz="0 0 0" rpy="0 0 0"/>
@@ -196,10 +196,10 @@
       </geometry>
     </collision>
-  </link>
-  <joint name="table_to_chessboard_joint" type="fixed">
-    <parent link="table_link"/>
-    <child link="chessboard_link"/>
-    <origin xyz="0 0 0.272" rpy="0 0 1.5708"/>
-  </joint>
+    </link>
+    <joint name="table_to_chessboard_joint" type="fixed">
+      <parent link="table_link"/>
+      <child link="chessboard_link"/>
+      <origin xyz="0 0 0.182" rpy="0 0 1.5708"/>
+    </joint>
   <!-- Gazebo - ROS 2 control -->
   <xacro:if value="$(arg ros2_control)">

Commit message: Second robot arm

File: panda_description/urdf/panda.urdf.xacro (robot description, xacro)
@@ -16,4 +16,7 @@
   <!-- Prefix for all entities -->
   <xacro:arg name="prefix" default="$(arg name)_"/>
+  <!-- Origin of the arm in the world -->
+  <xacro:arg name="origin_xyz" default="0 0 0"/>
+  <xacro:arg name="origin_rpy" default="0 0 0"/>
   <!-- Flag to enable default gripper -->
   <xacro:arg name="gripper" default="true" />
@@ -48,6 +51,6 @@
   <!-- Origin of arm in the world -->
   <xacro:property name="world_name" value="world"/>
-  <xacro:property name="origin_xyz" value="0 0 0"/>
-  <xacro:property name="origin_rpy" value="0 0 0"/>
+  <xacro:property name="origin_xyz" value="$(arg origin_xyz)"/>
+  <xacro:property name="origin_rpy" value="$(arg origin_rpy)"/>
   <!-- Offset of gripper with respect to wrist flange -->
   <xacro:property name="gripper_offset_xyz" value="0 0 0"/>
